File: Drehscheibe/Drehscheibe.kicad_sch (KiCad schematic)
At the start: 14 parts, among them J1 Raspberry_Pi_2_3, J2 Motor, J3 LCD_01, J4 LCD_02, J5 LED, J6 PSU, Q1 IRF8736, Q2 IRF8736

Commit message: new Version
Connections:
- net GND: now also J1.14 (GND), J1.20 (GND), J1.30 (GND), J1.34 (GND), J1.39 (GND), J1.6 (GND), J1.9 (GND)
Changed lines of the file:
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@@
     (rev "1.0")
+  )
+  (junction (at 67.31 147.32) (diameter 0) (color 0 0 0 0)
   )
   (junction (at 146.05 58.42) (diameter 0) (color 0 0 0 0)
   )
+  (junction (at 72.39 147.32) (diameter 0) (color 0 0 0 0)
+  )
+  (junction (at 62.23 147.32) (diameter 0) (color 0 0 0 0)
+  )
+  (junction (at 69.85 147.32) (diameter 0) (color 0 0 0 0)
+  )
+  (junction (at 64.77 147.32) (diameter 0) (color 0 0 0 0)
+  )
   (junction (at 146.05 50.8) (diameter 0) (color 0 0 0 0)
+  )
+  (junction (at 74.93 147.32) (diameter 0) (color 0 0 0 0)
   )
   (junction (at 64.77 81.28) (diameter 0) (color 0 0 0 0)
@@
     (stroke (width 0) (type default) (color 0 0 0 0))
   )
+  (wire (pts (xy 72.39 147.32) (xy 74.93 147.32))
+    (stroke (width 0) (type default) (color 0 0 0 0))
+  )
   (wire (pts (xy 194.31 49.53) (xy 194.31 48.26))
     (stroke (width 0) (type default) (color 0 0 0 0))
   )
   (wire (pts (xy 146.05 58.42) (xy 146.05 60.96))
+    (stroke (width 0) (type default) (color 0 0 0 0))
+  )
+  (wire (pts (xy 74.93 147.32) (xy 77.47 147.32))
     (stroke (width 0) (type default) (color 0 0 0 0))
   )
@@
     (stroke (width 0) (type default) (color 0 0 0 0))
   )
+  (wire (pts (xy 62.23 147.32) (xy 64.77 147.32))
+    (stroke (width 0) (type default) (color 0 0 0 0))
+  )
   (polyline (pts (xy 116.84 40.64) (xy 161.29 40.64))
     (stroke (width 0) (type default) (color 0 0 0 0))
   )
   (polyline (pts (xy 161.29 81.28) (xy 116.84 81.28))
+    (stroke (width 0) (type default) (color 0 0 0 0))
+  )
+  (wire (pts (xy 64.77 147.32) (xy 67.31 147.32))
     (stroke (width 0) (type default) (color 0 0 0 0))
   )
@@
     (stroke (width 0) (type default) (color 0 0 0 0))
   )
+  (wire (pts (xy 69.85 147.32) (xy 72.39 147.32))
+    (stroke (width 0) (type default) (color 0 0 0 0))
+  )
+  (wire (pts (xy 59.69 147.32) (xy 62.23 147.32))
+    (stroke (width 0) (type default) (color 0 0 0 0))
+  )
   (wire (pts (xy 146.05 48.26) (xy 146.05 50.8))
     (stroke (width 0) (type default) (color 0 0 0 0))
   )
+  (wire (pts (xy 67.31 147.32) (xy 69.85 147.32))
+    (stroke (width 0) (type default) (color 0 0 0 0))
+  )
